File: Kamaitachi.kicad_pcb (KiCad board)
At the start: 2 copper layers, 0 parts

Commit message: pcb in progress
Parts:
- added D1: 1N4148, Diode_SMD:D_SOD-123, B.Cu at (88.3, 121.0)
- added D10: 1N4148, Diode_SMD:D_SOD-123, B.Cu at (126.4, 153.8)
- added D11: 1N4148, Diode_SMD:D_SOD-123, B.Cu at (145.5, 113.3)
- added D12: 1N4148, Diode_SMD:D_SOD-123, B.Cu at (145.5, 132.4)
- added D13: 1N4148, Diode_SMD:D_SOD-123, B.Cu at (145.5, 151.4)
- added D14: 1N4148, Diode_SMD:D_SOD-123, B.Cu at (155.0, 175.3)
- added D15: 1N4148, Diode_SMD:D_SOD-123, B.Cu at (164.5, 118.1)
- added D16: 1N4148, Diode_SMD:D_SOD-123, B.Cu at (164.5, 137.2)
- added D17: 1N4148, Diode_SMD:D_SOD-123, B.Cu at (164.5, 156.2)
- added D18: 1N4148, Diode_SMD:D_SOD-123, B.Cu at (179.7, 179.2)
- added D19: 1N4148, Diode_SMD:D_SOD-123, B.Cu at (183.6, 118.1)
- added D2: 1N4148, Diode_SMD:D_SOD-123, B.Cu at (88.3, 140.0)
- added D20: 1N4148, Diode_SMD:D_SOD-123, B.Cu at (183.6, 137.2)
- added D21: 1N4148, Diode_SMD:D_SOD-123, B.Cu at (183.6, 156.2)
- added D22: 1N4148, Diode_SMD:D_SOD-123, B.Cu at (212.2, 161.0)
- added D23: 1N4148, Diode_SMD:D_SOD-123, B.Cu at (240.7, 118.1)
- added D24: 1N4148, Diode_SMD:D_SOD-123, B.Cu at (240.7, 137.2)
- added D25: 1N4148, Diode_SMD:D_SOD-123, B.Cu at (240.7, 156.2)
- added D26: 1N4148, Diode_SMD:D_SOD-123, B.Cu at (244.4, 176.6)
- added D27: 1N4148, Diode_SMD:D_SOD-123, B.Cu at (259.8, 118.1)
- added D28: 1N4148, Diode_SMD:D_SOD-123, B.Cu at (259.8, 137.2)
- added D29: 1N4148, Diode_SMD:D_SOD-123, B.Cu at (259.8, 156.2)
- added D3: 1N4148, Diode_SMD:D_SOD-123, B.Cu at (88.3, 159.1)
- added D30: 1N4148, Diode_SMD:D_SOD-123, B.Cu at (269.3, 175.3)
- added D31: 1N4148, Diode_SMD:D_SOD-123, B.Cu at (278.8, 113.3)
- added D32: 1N4148, Diode_SMD:D_SOD-123, B.Cu at (278.8, 132.4)
- added D33: 1N4148, Diode_SMD:D_SOD-123, B.Cu at (278.8, 151.4)
- added D34: 1N4148, Diode_SMD:D_SOD-123, B.Cu at (297.9, 115.7)
- added D35: 1N4148, Diode_SMD:D_SOD-123, B.Cu at (297.9, 134.8)
- added D36: 1N4148, Diode_SMD:D_SOD-123, B.Cu at (297.9, 153.8)
- added D37: 1N4148, Diode_SMD:D_SOD-123, B.Cu at (316.9, 121.0)
- added D38: 1N4148, Diode_SMD:D_SOD-123, B.Cu at (316.9, 140.0)
- added D39: 1N4148, Diode_SMD:D_SOD-123, B.Cu at (316.9, 159.1)
- added D4: 1N4148, Diode_SMD:D_SOD-123, B.Cu at (107.4, 121.0)
- added D40: 1N4148, Diode_SMD:D_SOD-123, B.Cu at (321.7, 178.1)
- added D41: 1N4148, Diode_SMD:D_SOD-123, B.Cu at (336.0, 121.0)
- added D42: 1N4148, Diode_SMD:D_SOD-123, B.Cu at (336.0, 140.0)
- added D43: 1N4148, Diode_SMD:D_SOD-123, B.Cu at (336.0, 159.1)
- added D5: 1N4148, Diode_SMD:D_SOD-123, B.Cu at (107.4, 140.0)
- added D6: 1N4148, Diode_SMD:D_SOD-123, B.Cu at (107.4, 159.1)
- added D7: 1N4148, Diode_SMD:D_SOD-123, B.Cu at (102.6, 178.1)
- added D8: 1N4148, Diode_SMD:D_SOD-123, B.Cu at (126.4, 115.7)
- added D9: 1N4148, Diode_SMD:D_SOD-123, B.Cu at (126.4, 134.8)
- added SW1: SW_PUSH, emptystring:CherryMX_Hotswap_Back, F.Cu at (83.3, 116.0)
- added SW10: SW_PUSH, emptystring:CherryMX_Hotswap_Back, F.Cu at (121.4, 148.8)
- added SW11: SW_PUSH, emptystring:CherryMX_Hotswap_Back, F.Cu at (140.5, 108.3)
- added SW12: SW_PUSH, emptystring:CherryMX_Hotswap_Back, F.Cu at (140.5, 127.4)
- added SW13: SW_PUSH, emptystring:CherryMX_Hotswap_Back, F.Cu at (140.5, 146.4)
- added SW14: SW_PUSH, emptystring:CherryMX_Hotswap_Back, F.Cu at (150.0, 170.3)
- added SW15: SW_PUSH, emptystring:CherryMX_Hotswap_Back, F.Cu at (159.5, 113.1)
- added SW16: SW_PUSH, emptystring:CherryMX_Hotswap_Back, F.Cu at (159.5, 132.2)
- added SW17: SW_PUSH, emptystring:CherryMX_Hotswap_Back, F.Cu at (159.5, 151.2)
- added SW18: SW_PUSH, emptystring:CherryMX_Hotswap_Back, F.Cu at (175.7, 173.4)
- added SW19: SW_PUSH, emptystring:CherryMX_Hotswap_Back, F.Cu at (178.6, 113.1)
- added SW2: SW_PUSH, emptystring:CherryMX_Hotswap_Back, F.Cu at (83.3, 135.0)
- added SW20: SW_PUSH, emptystring:CherryMX_Hotswap_Back, F.Cu at (178.6, 132.2)
- added SW21: SW_PUSH, emptystring:CherryMX_Hotswap_Back, F.Cu at (178.6, 151.2)
- added SW22: SW_PUSH, emptystring:CherryMX_Hotswap_Back, F.Cu at (207.2, 156.0)
- added SW23: SW_PUSH, emptystring:CherryMX_Hotswap_Back, F.Cu at (235.7, 113.1)
- added SW24: SW_PUSH, emptystring:CherryMX_Hotswap_Back, F.Cu at (235.7, 132.2)
- added SW25: SW_PUSH, emptystring:CherryMX_Hotswap_Back, F.Cu at (235.7, 151.2)
- added SW26: SW_PUSH, emptystring:CherryMX_Hotswap_Back, F.Cu at (238.6, 173.4)
- added SW27: SW_PUSH, emptystring:CherryMX_Hotswap_Back, F.Cu at (254.8, 113.1)
- added SW28: SW_PUSH, emptystring:CherryMX_Hotswap_Back, F.Cu at (254.8, 132.2)
- added SW29: SW_PUSH, emptystring:CherryMX_Hotswap_Back, F.Cu at (254.8, 151.2)
- added SW3: SW_PUSH, emptystring:CherryMX_Hotswap_Back, F.Cu at (83.3, 154.1)
- added SW30: SW_PUSH, emptystring:CherryMX_Hotswap_Back, F.Cu at (264.3, 170.3)
- added SW31: SW_PUSH, emptystring:CherryMX_Hotswap_Back, F.Cu at (273.8, 108.3)
- added SW32: SW_PUSH, emptystring:CherryMX_Hotswap_Back, F.Cu at (273.8, 127.4)
- added SW33: SW_PUSH, emptystring:CherryMX_Hotswap_Back, F.Cu at (273.8, 146.4)
- added SW34: SW_PUSH, emptystring:CherryMX_Hotswap_Back, F.Cu at (292.9, 110.7)
- added SW35: SW_PUSH, emptystring:CherryMX_Hotswap_Back, F.Cu at (292.9, 129.8)
- added SW36: SW_PUSH, emptystring:CherryMX_Hotswap_Back, F.Cu at (292.9, 148.8)
- added SW37: SW_PUSH, emptystring:CherryMX_Hotswap_Back, F.Cu at (311.9, 116.0)
- added SW38: SW_PUSH, emptystring:CherryMX_Hotswap_Back, F.Cu at (311.9, 135.0)
- added SW39: SW_PUSH, emptystring:CherryMX_Hotswap_Back, F.Cu at (311.9, 154.1)
- added SW4: SW_PUSH, emptystring:CherryMX_Hotswap_Back, F.Cu at (102.4, 116.0)
- added SW40: SW_PUSH, emptystring:CherryMX_Hotswap_Back, F.Cu at (316.7, 173.1)
- added SW41: SW_PUSH, emptystring:CherryMX_Hotswap_Back, F.Cu at (331.0, 116.0)
- added SW42: SW_PUSH, emptystring:CherryMX_Hotswap_Back, F.Cu at (331.0, 135.0)
- added SW43: SW_PUSH, emptystring:CherryMX_Hotswap_Back, F.Cu at (331.0, 154.1)
- added SW44: SW_PUSH, kbd:ResetSW, F.Cu at (207.2, 134.5)
- added SW5: SW_PUSH, emptystring:CherryMX_Hotswap_Back, F.Cu at (102.4, 135.0)
- added SW6: SW_PUSH, emptystring:CherryMX_Hotswap_Back, F.Cu at (102.4, 154.1)
- added SW7: SW_PUSH, emptystring:CherryMX_Hotswap_Back, F.Cu at (97.6, 173.1)
- added SW8: SW_PUSH, emptystring:CherryMX_Hotswap_Back, F.Cu at (121.4, 110.7)
- added SW9: SW_PUSH, emptystring:CherryMX_Hotswap_Back, F.Cu at (121.4, 129.8)
- added U1: ProMicro, emptystring:ProMicro_v2_Backside, F.Cu at (207.2, 114.3)
Routing:
- net col4: track 0.00 -> 66.1 mm
- net col3: track 0.00 -> 65.9 mm
- net col6: track 0.00 -> 62.6 mm
- net col7: track 0.00 -> 61.2 mm
- net col10: track 0.00 -> 59.2 mm
- net col1: track 0.00 -> 59.2 mm
- net col9: track 0.00 -> 38.1 mm
- net col2: track 0.00 -> 38.1 mm
- net col5: track 0.00 -> 38.1 mm
- net col8: track 0.00 -> 38.1 mm
- net col11: track 0.00 -> 38.1 mm
- net col0: track 0.00 -> 38.1 mm
- net row2: track 0.00 -> 20.5 mm, vias 0 -> 2
- net row1: track 0.00 -> 20.5 mm, vias 0 -> 2
- net row0: track 0.00 -> 20.5 mm, vias 0 -> 2
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- added copper zone on B.Cu, net GND
- added copper zone on F.Cu, net GND
Other:
- board outline added: 271.5 x 96.4 mm

Commit message: pcb finished
Parts:
- SW1, SW10, SW11, SW12, SW13, SW14, SW15, SW16, SW17, SW19, SW2, SW20, SW21, SW22, SW23, SW24, SW25, SW27, SW28, SW29, SW3, SW30, SW31, SW32, SW33, SW34, SW35, SW36, SW37, SW38, SW39, SW4, SW41, SW42, SW43, SW5, SW6, SW8, SW9: footprint emptystring:CherryMX_Hotswap_Back -> Keebio-Parts:MX_PCB_100H
- SW18, SW26: footprint emptystring:CherryMX_Hotswap_Back -> Keebio-Parts:MX_PCB_125H
- SW40, SW7: footprint emptystring:CherryMX_Hotswap_Back -> Keebio-Parts:MX_PCB_150H
- U1: moved to B.Cu
- moved D18 5.37 mm to (176.3, 183.3), turned to 165 degrees
- moved D19 5.03 mm to (185.4, 122.8), turned to 175 degrees
- moved D41 4.93 mm to (334.0, 116.5), turned to 185 degrees
- moved SW19 4.84 mm to (180.9, 117.4), turned to 355 degrees
- moved SW23 4.84 mm to (233.4, 117.4), turned to 5 degrees
- moved D43 4.84 mm to (337.3, 154.4), turned to 185 degrees
- moved SW26 4.79 mm to (241.5, 177.2), turned to 15 degrees
- moved SW18 4.79 mm to (172.8, 177.2), turned to 345 degrees
- moved D21 4.76 mm to (182.1, 160.7), turned to 175 degrees
- moved SW1 4.72 mm to (85.8, 111.9), turned to 355 degrees
- moved SW41 4.72 mm to (328.6, 111.9), turned to 5 degrees
- moved D40 4.62 mm to (324.7, 174.6), turned to 185 degrees
- moved D20 4.61 mm to (183.8, 141.8), turned to 175 degrees
- moved D42 4.59 mm to (335.7, 135.4), turned to 185 degrees
- moved D26 4.57 mm to (247.6, 179.9), turned to 195 degrees
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Connections:
- U1 pad 10: col11 -> col5
- U1 pad 11: row2 -> row0
- U1 pad 12: row3 -> row1
- U1 pad 13: col5 -> row3
- U1 pad 14: col4 -> row2
- U1 pad 15: col3 -> col6
- U1 pad 16: col2 -> col7
- U1 pad 17: col1 -> col8
- U1 pad 18: col0 -> col9
- U1 pad 19: row1 -> col10
- U1 pad 20: row0 -> col11
- U1 pad 5: col6 -> col0
- U1 pad 6: col7 -> col1
- U1 pad 7: col8 -> col2
- U1 pad 8: col9 -> col3
- U1 pad 9: col10 -> col4
Routing:
- net row2: track 20.5 -> 357.0 mm, vias 2 -> 1
- net row3: track 0.00 -> 318.9 mm, vias 0 -> 2
- net row1: track 20.5 -> 317.3 mm, vias 2 -> 0
- net row0: track 20.5 -> 306.0 mm, vias 2 -> 0
- net col11: track 38.1 -> 171.2 mm
- net col0: track 38.1 -> 164.6 mm
- net col10: track 59.2 -> 174.9 mm
- net col1: track 59.2 -> 169.9 mm
- net col9: track 38.1 -> 131.4 mm
- net col2: track 38.1 -> 127.9 mm
- net col8: track 38.1 -> 110.3 mm
- net col3: track 65.9 -> 135.8 mm
- net col5: track 38.1 -> 106.4 mm
- net col7: track 61.2 -> 120.8 mm
- net col4: track 66.1 -> 125.6 mm
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Other:
- board size 271.5 x 96.4 mm -> 271.5 x 100 mm
